File: Circuito de corriente.kicad_pcb (KiCad board)
At the start: 2 copper layers, 150 x 120 mm, 111 parts, among them J1 SALIDAS, J2 ENTRADAS, J3 +12V2, J4 +3V3, J5 +/- 5V, J6 +/- 12V, J7 INPUT_CEDCp, K1 JJM1-12V, K2 JJM1-12V, K3 JJM1-12V, K4 SLA-12VDC-SL-C, M1 Fan_3pin, Q1 BC337, Q2 BC327, U1 OPA604, U13 LM35-NEB, U16 Fuse, U18 IRLZ44N, U2 OPA604, U20 IRLZ44N, U22 IRLZ44N, U3 A6841, U4 AD7606_M, U5 MCP4725, U55 IRLZ44N, U6 OPA604, U7 OPA604, U8 OPA604

Commit message: V4 Ltspice
Parts:
- removed the C13 at (206.7, 126.1)
- removed J7: INPUT_CEDCp, CEDCp:Bornera_1x4
- removed R19: 22k, CEDCp:Resistencia_0,25W
- removed the R20 at (144.6, 94.1)
- removed the R21 at (144.6, 90.5)
- removed the R22 at (144.6, 86.9)
- removed REF**: KiCad-Logo2_5mm_SilkScreen, Symbol:KiCad-Logo2_5mm_SilkScreen
- removed REF**: OSHW-Logo_5.7x6mm_SilkScreen, Symbol:OSHW-Logo_5.7x6mm_SilkScreen
- removed the U4 at (150.1, 114.2)
- removed U7: OPA604, CEDCp:OPA604
- added C7: 10u, Capacitor_THT:CP_Radial_D4.0mm_P2.00mm, F.Cu at (143.4, 144.4)
- added J11: Conn_01x01, Connector_Wire:SolderWire-2sqmm_1x01_D2mm_OD3.9mm, F.Cu at (214.2, 52.3)
- added J12: Conn_01x01, Connector_Wire:SolderWire-0.5sqmm_1x01_D0.9mm_OD2.3mm, F.Cu at (124.9, 156.7)
- added J13: Conn_01x01, Connector_Wire:SolderWire-2sqmm_1x01_D2mm_OD3.9mm, F.Cu at (214.2, 61.3)
- added J14: Conn_01x01, Connector_Wire:SolderWire-0.5sqmm_1x01_D0.9mm_OD2.3mm, F.Cu at (129.8, 156.7)
- added R11: 22k, CEDCp_V2:Resistencia_0,25W, F.Cu at (98.8, 30.5)
- added R16: 22k, CEDCp_V2:Resistencia_0,25W, F.Cu at (98.8, 38.5)
- added R17: 22k, CEDCp_V2:Resistencia_0,25W, F.Cu at (98.8, 46.0)
- added R8: 22k, CEDCp_V2:Resistencia_0,25W, F.Cu at (98.8, 22.5)
- added U26: MCP4725_Placa, CEDCp_V2:MCP4725_Placa, F.Cu at (160.3, 135.3)
- added UB2: AD7606_M, CEDCp_V2:AD7606_M, F.Cu at (166.8, 156.9)
- D5: renamed from D1; footprint Diode_THT:D_DO-15_P10.16mm_Horizontal -> Diode_THT:D_DO-41_SOD81_P10.16mm_Horizontal
- Q61: renamed from Q1; footprint CEDCp:BC548 -> Package_TO_SOT_THT:TO-92_Inline
- Q62: renamed from Q2; footprint CEDCp:BC548 -> Package_TO_SOT_THT:TO-92_Inline
- R10: renamed from R8; footprint CEDCp:Resistencia_0,25W -> CEDCp_V2:Resistencia_0,25W
- R13: renamed from R29; footprint CEDCp:Resistencia_0,25W -> CEDCp_V2:Resistencia_0,25W
- R14: renamed from R4; footprint CEDCp:Resistencia_0,25W -> CEDCp_V2:Resistencia_0,25W
- R15: renamed from R30; footprint CEDCp:Resistencia_0,25W -> CEDCp_V2:Resistencia_0,25W
- R18: renamed from R28; footprint CEDCp:Resistencia_0,25W -> CEDCp_V2:Resistencia_0,25W
- R20: renamed from R10; footprint CEDCp:Resistencia_0,25W -> CEDCp_V2:Resistencia_0,25W
- R21: renamed from R18; footprint CEDCp:Resistencia_0,25W -> CEDCp_V2:Resistencia_0,25W
- R23, R5, ROp1, ROp2, ROp3, ROp4: footprint CEDCp:Resistencia_0,25W -> CEDCp_V2:Resistencia_0,25W
- R24: renamed from R15; footprint CEDCp:Resistencia_0,25W -> CEDCp_V2:Resistencia_0,25W
- R25: renamed from R16; footprint CEDCp:Resistencia_0,25W -> CEDCp_V2:Resistencia_0,25W
- R26: renamed from R24; footprint CEDCp:Resistencia_0,25W -> CEDCp_V2:Resistencia_0,25W
- R27: renamed from R17; footprint CEDCp:Resistencia_0,25W -> CEDCp_V2:Resistencia_0,25W
- R29: renamed from R31; footprint CEDCp:Resistencia_0,25W -> CEDCp_V2:Resistencia_0,25W
- R3: renamed from R7; footprint CEDCp:Resistencia_0,25W -> CEDCp_V2:Resistencia_0,25W
- R30: renamed from R12; footprint CEDCp:Resistencia_0,25W -> CEDCp_V2:Resistencia_0,25W
- R31: renamed from R32; footprint CEDCp:Resistencia_0,25W -> CEDCp_V2:Resistencia_0,25W
- R33: renamed from R39; footprint CEDCp:Resistencia_0,25W -> CEDCp_V2:Resistencia_0,25W
- R34: renamed from R33; footprint CEDCp:Resistencia_0,25W -> CEDCp_V2:Resistencia_0,25W
- R35: renamed from R34; footprint CEDCp:Resistencia_0,25W -> CEDCp_V2:Resistencia_0,25W
- R36: renamed from R35; footprint CEDCp:Resistencia_0,25W -> CEDCp_V2:Resistencia_0,25W
- R37: renamed from R36; footprint CEDCp:Resistencia_0,25W -> CEDCp_V2:Resistencia_0,25W
- R38: renamed from R25; footprint CEDCp:Resistencia_0,25W -> CEDCp_V2:Resistencia_0,25W
- R39: renamed from R26; footprint CEDCp:Resistencia_0,25W -> CEDCp_V2:Resistencia_0,25W
- R4: renamed from R3; footprint CEDCp:Resistencia_0,25W -> CEDCp_V2:Resistencia_0,25W
- R40: renamed from R13; footprint CEDCp:Resistencia_0,25W -> CEDCp_V2:Resistencia_0,25W
- R41: renamed from R38; footprint CEDCp:Resistencia_0,25W -> CEDCp_V2:Resistencia_0,25W
- R43: renamed from R27; footprint CEDCp:Resistencia_0,25W -> CEDCp_V2:Resistencia_0,25W
- R6: renamed from R1; footprint CEDCp:Resistencia_0,25W -> CEDCp_V2:Resistencia_0,25W
- R7: renamed from R6; footprint CEDCp:Resistencia_0,25W -> CEDCp_V2:Resistencia_0,25W
- R9: renamed from R2; footprint CEDCp:Resistencia_0,25W -> CEDCp_V2:Resistencia_0,25W
- U5: value MCP4725 -> OPA604; footprint Connector_PinHeader_2.54mm:PinHeader_1x06_P2.54mm_Vertical -> CEDCp:OPA604
- UA1, UA2, UA3, UA4, UA5: value LM311 -> LM311_V2; footprint CEDCp:LM311P -> CEDCp_V2:LM311_V2
- moved J3 142.5 mm to (213.8, 85.0), turned to -90 degrees
- moved U25 125.8 mm to (215.3, 98.4)
- moved RV4 112.5 mm to (85.0, 150.5)
- moved D8 112.1 mm to (81.2, 138.8), turned to 0 degrees
- moved RV5 109.2 mm to (75.6, 141.8), turned to 90 degrees
- moved U5 104.6 mm to (102.0, 139.8), turned to 0 degrees
- moved R43 103.6 mm to (86.3, 144.7)
- moved RV9 102.4 mm to (182.5, 66.3), turned to 90 degrees
- moved J5 89.9 mm to (151.5, 156.1), turned to 180 degrees
- moved R24 88.9 mm to (87.1, 80.9), turned to 180 degrees
- moved J1 88.4 mm to (215.2, 153.1), turned to 180 degrees
- moved R13 86.3 mm to (103.1, 152.3)
- moved C5 86.3 mm to (86.1, 55.1), turned to -90 degrees
- moved R21 86.3 mm to (82.3, 68.4)
- moved R18 86.1 mm to (103.2, 148.5), turned to 0 degrees
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- renumbered C5 to C1, C14 to C11, C2 to C13, C1 to C15, C8 to C2, C7 to C28, C6 to C29, C11 to C30, C10 to C31, C9 to C4, C4 to C5, C12 to C6, C15 to C9, D2 to D8, R9 to R12, R11 to R22, R37 to R32, R14 to R42, U55 to U1, U6 to U11, U16 to U19, U18 to U2, U8 to U20, U13 to U25, U20 to U3, U22 to U4, U1 to U6, U2 to U60, U3 to UB1, UB1 to UB3
Connections:
- J1 pad 10: /toMicroC_ADC_BUSY -> /toMicroC_OverVoltageSignal
- J1 pad 9: /toMicroC_OverVoltageSignal -> /toMicroC_ADC_BUSY
- J3 pad 1: /+12V2 -> GND
- J3 pad 2: GND -> /+12V2
- J5 pad 1: /+5V -> /-5V
- J5 pad 3: /-5V -> /+5V
- K1 pad 3: /PushPullOut -> GND
- K1 pad 4: GND -> /PushPullOut
- K2 pad 3: /PushPullOut -> GND
- K2 pad 4: GND -> /PushPullOut
- K3 pad 3: /PushPullOut -> GND
- K3 pad 4: GND -> /PushPullOut
- Q62 pad 1: /PushPullOut -> /-12V
- Q62 pad 3: /-12V -> /PushPullOut
- R13 pad 2: Net-(R28-Pad2) -> Net-(R13-Pad2)
- R15 pad 1: Net-(R28-Pad2) -> Net-(R13-Pad2)
- R18 pad 2: Net-(R28-Pad2) -> Net-(R13-Pad2)
- U11 pad 6: unconnected-(U6-Pad6) -> /Error1
- U5 pad 1: /fromDAC_Vref -> Net-(RV7-Pad3)
- U5 pad 2: GND -> Net-(R13-Pad2)
- U5 pad 3: /+3.3V -> /Lazo Realimentacion de Voltaje (Lazo 2)/1.1V
- U5 pad 4: /fromMicroC_DACI2C_SDA -> /-12V
- U5 pad 5: /fromMicroC_DACI2C_SCL -> Net-(RV7-Pad1)
- U5 pad 6: GND -> /Error2
Routing:
- net GND: track 46.1 -> 1159.8 mm, vias 1 -> 4
- net /fromA6841_FeedbackLoopSelection: track 261.4 -> 70.1 mm, vias 2 -> 1
- net /toADC_LoadCurrent: track 60.1 -> 229.9 mm
- net /fromDAC_Vref: track 76.3 -> 194.6 mm, vias 0 -> 2
- net /CEP_Input+_MOS: track 0.00 -> 110.9 mm
- net /toMicroC_OverVoltageSignal: track 140.7 -> 30.7 mm, vias 1 -> 0
- net /+12V2: track 247.2 -> 171.3 mm, vias 0 -> 2
- net /fromA6841_PowerEnable: track 23.9 -> 99.3 mm, vias 0 -> 1
- net /fromMicroC_A6841ST1: track 10.6 -> 83.6 mm, vias 0 -> 1
- net /fromMicroC_DACI2C_SDA: track 6.55 -> 74.6 mm
- net /fromMicroC_DACI2C_SCL: track 6.55 -> 70.6 mm
- net /fromMicroC_A6841CLK1: track 24.0 -> 85.8 mm
- net /ILimit_Vref: track 144.6 -> 83.6 mm, vias 4 -> 5
- net /toADC_LoadVoltage: track 100.6 -> 161.2 mm, vias 2 -> 0
- net /fromMicroC_A6841SerialDataIN: track 35.3 -> 87.9 mm
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- added copper zone on F.Cu, net /CEP_Input+_MOS
- removed copper zone on B.Cu, net /CEP_Input+_MOS
Other:
- board size 150 x 120 mm -> 150 x 148.2 mm
- board text added: "Hay conexiones de mas debido a que si insertamos los planos a maza eso se evitaria"
- board text added: "No coincidian las esquinas de EDGE CUTS"
- board text removed: "Módulo de potencia"
