File: Circuito de corriente.kicad_sch (KiCad schematic)
At the start: 6 parts, among them J1 SALIDAS, J2 ENTRADAS

Commit message: Reorder conection with control module
Connections:
- net fromMicroC_ADC_CONV: now also J2.3 (Pin_3); no longer J2.5 (Pin_5)
- net fromMicroC_ADC_RD: now also J2.1 (Pin_1); no longer J2.3 (Pin_3)
- net fromMicroC_ADC_RST: now also J2.2 (Pin_2); no longer J2.4 (Pin_4)
- net fromMicroC_DACI2C_SCL: now also J2.4 (Pin_4); no longer J2.2 (Pin_2)
- net fromMicroC_DACI2C_SDA: now also J2.5 (Pin_5); no longer J2.1 (Pin_1)
- net toMicroC_ADC_BUSY: now also J1.10 (Pin_10); no longer J1.2 (Pin_2)
- net toMicroC_ADC_DB0: now also J1.1 (Pin_1); no longer J1.3 (Pin_3)
- net toMicroC_ADC_DB1: now also J1.2 (Pin_2); no longer J1.4 (Pin_4)
- net toMicroC_ADC_DB2: now also J1.3 (Pin_3); no longer J1.5 (Pin_5)
- net toMicroC_ADC_DB3: now also J1.4 (Pin_4); no longer J1.6 (Pin_6)
- net toMicroC_ADC_DB4: now also J1.5 (Pin_5); no longer J1.7 (Pin_7)
- net toMicroC_ADC_DB5: now also J1.6 (Pin_6); no longer J1.8 (Pin_8)
- net toMicroC_ADC_DB6: now also J1.7 (Pin_7); no longer J1.9 (Pin_9)
- net toMicroC_ADC_DB7: now also J1.8 (Pin_8); no longer J1.10 (Pin_10)
- net toMicroC_OverVoltageSignal: now also J1.9 (Pin_9); no longer J1.1 (Pin_1)
Changed lines of the file:
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@@
     (effects (font (size 1.27 1.27) bold) (justify left bottom))
   )
-  (label "toMicroC_ADC_DB6" (at 116.84 185.42 180)
+  (label "toMicroC_ADC_DB6" (at 116.84 180.34 180)
     (effects (font (size 1.27 1.27) (thickness 0.254) bold) (justify right bottom))
   )
@@
     (effects (font (size 1.27 1.27) bold) (justify right bottom))
   )
-  (label "toMicroC_ADC_BUSY" (at 116.84 167.64 180)
+  (label "toMicroC_ADC_BUSY" (at 116.84 187.96 180)
     (effects (font (size 1.27 1.27) (thickness 0.254) bold) (justify right bottom))
   )
@@
     (effects (font (size 1.27 1.27) bold) (justify right bottom))
   )
-  (label "toMicroC_ADC_DB7" (at 116.84 187.96 180)
+  (label "toMicroC_ADC_DB7" (at 116.84 182.88 180)
     (effects (font (size 1.27 1.27) (thickness 0.254) bold) (justify right bottom))
   )
@@
     (effects (font (size 1.27 1.27) (thickness 0.254) bold) (justify left bottom))
   )
-  (label "fromMicroC_ADC_RST" (at 139.573 172.72 0)
+  (label "fromMicroC_ADC_RST" (at 139.573 167.64 0)
     (effects (font (size 1.27 1.27) (thickness 0.254) bold) (justify left bottom))
   )
@@
     (effects (font (size 1.27 1.27) bold) (justify right bottom))
   )
-  (label "toMicroC_ADC_DB5" (at 116.84 182.88 180)
-    (effects (font (size 1.27 1.27) (thickness 0.254) bold) (justify right bottom))
-  )
-  (label "toMicroC_ADC_DB1" (at 116.84 172.72 180)
+  (label "toMicroC_ADC_DB5" (at 116.84 177.8 180)
+    (effects (font (size 1.27 1.27) (thickness 0.254) bold) (justify right bottom))
+  )
+  (label "toMicroC_ADC_DB1" (at 116.84 167.64 180)
     (effects (font (size 1.27 1.27) (thickness 0.254) bold) (justify right bottom))
   )
@@
     (effects (font (size 1.27 1.27) bold) (justify left bottom))
   )
-  (label "fromMicroC_DACI2C_SCL" (at 139.573 167.64 0)
+  (label "fromMicroC_DACI2C_SCL" (at 139.573 172.72 0)
     (effects (font (size 1.27 1.27) (thickness 0.254) bold) (justify left bottom))
   )
@@
     (effects (font (size 1.27 1.27) bold) (justify left bottom))
   )
-  (label "fromMicroC_ADC_CONV" (at 139.573 175.26 0)
-    (effects (font (size 1.27 1.27) (thickness 0.254) bold) (justify left bottom))
-  )
-  (label "toMicroC_ADC_DB2" (at 116.84 175.26 180)
+  (label "fromMicroC_ADC_CONV" (at 139.573 170.18 0)
+    (effects (font (size 1.27 1.27) (thickness 0.254) bold) (justify left bottom))
+  )
+  (label "toMicroC_ADC_DB2" (at 116.84 170.18 180)
     (effects (font (size 1.27 1.27) (thickness 0.254) bold) (justify right bottom))
   )
@@
     (effects (font (size 1.27 1.27) bold) (justify left bottom))
   )
-  (label "fromMicroC_ADC_RD" (at 139.573 170.18 0)
+  (label "fromMicroC_ADC_RD" (at 139.573 165.1 0)
     (effects (font (size 1.27 1.27) (thickness 0.254) bold) (justify left bottom))
   )
@@
     (effects (font (size 1.27 1.27) (thickness 0.254) bold) (justify left bottom))
   )
-  (label "toMicroC_ADC_DB4" (at 116.84 180.34 180)
+  (label "toMicroC_ADC_DB4" (at 116.84 175.26 180)
     (effects (font (size 1.27 1.27) (thickness 0.254) bold) (justify right bottom))
   )
@@
     (effects (font (size 1.27 1.27) (thickness 0.254) bold) (justify left bottom))
   )
-  (label "toMicroC_ADC_DB0" (at 116.84 170.18 180)
+  (label "toMicroC_ADC_DB0" (at 116.84 165.1 180)
     (effects (font (size 1.27 1.27) (thickness 0.254) bold) (justify right bottom))
   )
@@
     (effects (font (size 1.27 1.27) bold) (justify right bottom))
   )
-  (label "toMicroC_OverVoltageSignal" (at 116.84 165.1 180)
+  (label "toMicroC_OverVoltageSignal" (at 116.84 185.42 180)
     (effects (font (size 1.27 1.27) (thickness 0.254) bold) (justify right bottom))
   )
@@
     (effects (font (size 1.27 1.27) bold) (justify left bottom))
   )
-  (label "toMicroC_ADC_DB3" (at 116.84 177.8 180)
+  (label "toMicroC_ADC_DB3" (at 116.84 172.72 180)
     (effects (font (size 1.27 1.27) (thickness 0.254) bold) (justify right bottom))
   )
@@
     (effects (font (size 1.27 1.27) (thickness 0.254) bold) (justify right bottom))
   )
-  (label "fromMicroC_DACI2C_SDA" (at 139.573 165.1 0)
+  (label "fromMicroC_DACI2C_SDA" (at 139.573 175.26 0)
     (effects (font (size 1.27 1.27) (thickness 0.254) bold) (justify left bottom))
   )
@@
       (reference "J6") (unit 1) (value "+/- 12V") (footprint "CEDCp:Bornera_1x3")
     )
-    (path "/00000000-0000-0000-0000-00006277bc66/d7b48e3e-35a1-49dd-bccf-e336a4f4eb0a"
-      (reference "J7") (unit 1) (value "INPUT_CEDCp") (footprint "CEDCp:Bornera_1x2")
+    (path "/00000000-0000-0000-0000-00006277bc66/6613158f-59c2-473f-aaf3-c44415918fae"
+      (reference "J7") (unit 1) (value "INPUT_CEDCp") (footprint "CEDCp:Bornera_1x4")
     )
     (path "/00000000-0000-0000-0000-000061ae72e1/1da302e1-a7e5-4cbf-a296-61ecd8ff30a3"

Commit message: Gerbers generated again
Other:
- sheet Entrada_Alimentacion ports: added CEP_Inpunt+_1, CEP_Inpunt+_2; removed CEP_In(+)

Commit message: Pads mas grandes y correccion de vias
Other:
- sheet Adaptación_Señal_Control ports: added fromA6841_FeedbackLoopSelection; removed fromMicroC_FeedbackLoopSelection
- sheet Circuito de control de corriente ports: added CEP_Input+_MOS; removed CEP_Input+
- sheet Temperatura-Referencia-Fan ports: added fromA6841_toFanEnable; removed fromA6841_FanControl
Changed lines of the file:
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@@
     (effects (font (size 1.27 1.27) bold) (justify right bottom))
-  )
-  (label "fromMicroC_FBLSelection" (at 202.692 97.536 180)
-    (effects (font (size 1.27 1.27) (thickness 0.254) bold) (justify right bottom))
   )
   (label "-5V" (at 68.0212 42.291 0)
@@
   )
   (label "fromA6841_PowerEnable" (at 113.665 32.004 180)
+    (effects (font (size 1.27 1.27) (thickness 0.254) bold) (justify right bottom))
+  )
+  (label "fromA6841_FeedbackLoopSelection" (at 202.692 97.536 180)
     (effects (font (size 1.27 1.27) (thickness 0.254) bold) (justify right bottom))
   )
@@
       (effects (font (size 1.2954 1.2954)) (justify left))
     )
-    (pin "fromA6841_FanControl" input (at 43.688 173.355 180)
-      (effects (font (size 1.27 1.27)) (justify left))
-    )
     (pin "+12V2" input (at 70.358 181.483 0)
       (effects (font (size 1.27 1.27)) (justify right))
     )
     (pin "ILimint_Vref" output (at 43.688 176.911 180)
+      (effects (font (size 1.27 1.27)) (justify left))
+    )
+    (pin "fromA6841_toFanEnable" input (at 43.688 173.355 180)
       (effects (font (size 1.27 1.27)) (justify left))
     )
@@
       (effects (font (size 1.27 1.27)) (justify right))
     )
-    (pin "CEP_Input+" input (at 260.096 54.991 0)
-      (effects (font (size 1.27 1.27)) (justify right))
-    )
     (pin "+3.3V" input (at 260.096 32.512 0)
       (effects (font (size 1.27 1.27)) (justify right))
@@
     )
     (pin "V04" output (at 260.096 51.689 0)
+      (effects (font (size 1.27 1.27)) (justify right))
+    )
+    (pin "CEP_Input+_MOS" input (at 260.096 54.991 0)
       (effects (font (size 1.27 1.27)) (justify right))
     )
@@
       (effects (font (size 1.27 1.27)) (justify left top) hide)
     )
-    (pin "fromMicroC_FeedbackLoopSelection" input (at 203.708 97.536 180)
-      (effects (font (size 1.2954 1.2954)) (justify left))
-    )
     (pin "-5V" input (at 203.708 106.426 180)
       (effects (font (size 1.2954 1.2954)) (justify left))
@@
     (pin "-12V" input (at 241.427 110.236 0)
       (effects (font (size 1.27 1.27)) (justify right))
+    )
+    (pin "fromA6841_FeedbackLoopSelection" input (at 203.708 97.536 180)
+      (effects (font (size 1.27 1.27)) (justify left))
     )
   )
@@
       (reference "K1") (unit 1) (value "JJM1-12V") (footprint "CEDCp:RELAY_JJM1-12V")
     )
-    (path "/00000000-0000-0000-0000-000061ae72e1/28b61907-8b50-4d7e-a5f4-58682aa41ead"
+    (path "/00000000-0000-0000-0000-000061ae72e1/0946d05a-ca34-463c-99a2-e38f13436057"
       (reference "K2") (unit 1) (value "JJM1-12V") (footprint "CEDCp:RELAY_JJM1-12V")
     )
-    (path "/00000000-0000-0000-0000-000061ae72e1/a105f9af-b6c9-4bf3-8f84-efb2bdea968b"
+    (path "/00000000-0000-0000-0000-000061ae72e1/a2d8a91f-e909-4358-bc3e-7981fb94e6c3"
       (reference "K3") (unit 1) (value "JJM1-12V") (footprint "CEDCp:RELAY_JJM1-12V")
     )
@@
     )
     (path "/00000000-0000-0000-0000-000061a1268d/00000000-0000-0000-0000-000061a298f8"
-      (reference "U16") (unit 1) (value "Fuse") (footprint "Fuse:Fuse_Littelfuse-LVR100")
+      (reference "U16") (unit 1) (value "Fuse") (footprint "CEDCp:Fuse")
     )
     (path "/00000000-0000-0000-0000-000061ae72e1/00000000-0000-0000-0000-000061c87b47"

Commit message: V4 Ltspice
Parts:
- added HA1, HA2: MountingHole, MountingHole:MountingHole_2.2mm_M2_Pad_Via, symbol Mechanical:MountingHole
Connections:
- net toMicroC_ADC_BUSY: now also J1.9 (Pin_9); no longer J1.10 (Pin_10)
- net toMicroC_OverVoltageSignal: now also J1.10 (Pin_10); no longer J1.9 (Pin_9)
