File: Conversor_Analógico_Digital_3canales.kicad_sch (KiCad schematic)
At the start: 1 part, among them U4 AD7606_M

Commit message: Version V1 (Clearence + pads)
Connections:
- net GND: no longer U4.27 (CVB)
- net fromMicroC_ADC_CONV: now also U4.27 (CVB)
- no-connect marks 0 -> 7
Changed lines of the file:
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@@
 (kicad_sch (version 20211123) (generator eeschema)
   (paper "A4")
+  (junction (at 97.0026 86.5124) (diameter 0) (color 0 0 0 0)
+  )
   (junction (at 199.7964 91.7448) (diameter 0) (color 0 0 0 0)
   )
@@
   (junction (at 176.3776 94.2848) (diameter 0) (color 0 0 0 0)
   )
+  (junction (at 176.3776 83.8708) (diameter 0) (color 0 0 0 0)
+  )
   (junction (at 176.3776 91.7448) (diameter 0) (color 0 0 0 0)
   )
@@
   (junction (at 176.3776 89.2048) (diameter 0) (color 0 0 0 0)
   )
-  (junction (at 97.0026 96.6724) (diameter 0) (color 0 0 0 0)
+  (junction (at 199.7964 83.8708) (diameter 0) (color 0 0 0 0)
   )
   (junction (at 97.0026 89.0524) (diameter 0) (color 0 0 0 0)
   )
-  (junction (at 199.7964 83.8708) (diameter 0) (color 0 0 0 0)
+  (junction (at 94.742 119.5324) (diameter 0) (color 0 0 0 0)
+  )
+  (junction (at 95.0722 91.5924) (diameter 0) (color 0 0 0 0)
+  )
+  (junction (at 132.8166 71.7804) (diameter 0) (color 0 0 0 0)
   )
   (junction (at 176.3776 102.4128) (diameter 0) (color 0 0 0 0)
@@
   (junction (at 132.8166 83.9724) (diameter 0) (color 0 0 0 0)
   )
-  (junction (at 132.8166 86.5124) (diameter 0) (color 0 0 0 0)
-  )
   (junction (at 176.3776 86.4108) (diameter 0) (color 0 0 0 0)
   )
+  (no_connect (at 99.4156 111.9124))
+  (no_connect (at 99.4156 114.4524))
+  (no_connect (at 99.4156 116.9924))
+  (no_connect (at 129.8956 116.9924))
+  (no_connect (at 129.8956 111.9124))
+  (no_connect (at 129.8956 114.4524))
+  (no_connect (at 129.8956 99.2124))
+  (wire (pts (xy 132.0038 125.2982) (xy 132.0038 119.5324))
+    (stroke (width 0) (type default) (color 0 0 0 0))
+  )
   (wire (pts (xy 176.3776 97.0788) (xy 176.3776 99.8728))
     (stroke (width 0) (type default) (color 0 0 0 0))
   )
-  (wire (pts (xy 129.8956 91.5924) (xy 132.8166 91.5924))
+  (wire (pts (xy 129.8956 91.5924) (xy 136.7028 91.5924))
     (stroke (width 0) (type default) (color 0 0 0 0))
   )
@@
     (stroke (width 0) (type default) (color 0 0 0 0))
   )
+  (wire (pts (xy 132.0038 119.5324) (xy 129.8956 119.5324))
+    (stroke (width 0) (type default) (color 0 0 0 0))
+  )
   (wire (pts (xy 196.85 86.4108) (xy 199.7964 86.4108))
     (stroke (width 0) (type default) (color 0 0 0 0))
   )
+  (wire (pts (xy 94.742 119.5324) (xy 94.742 125.349))
+    (stroke (width 0) (type default) (color 0 0 0 0))
+  )
+  (wire (pts (xy 94.742 119.5324) (xy 99.4156 119.5324))
+    (stroke (width 0) (type default) (color 0 0 0 0))
+  )
   (wire (pts (xy 176.3776 89.2048) (xy 176.3776 91.7448))
     (stroke (width 0) (type default) (color 0 0 0 0))
@@
     (stroke (width 0) (type default) (color 0 0 0 0))
   )
-  (wire (pts (xy 97.0026 96.6724) (xy 97.0026 127.7874))
-    (stroke (width 0) (type default) (color 0 0 0 0))
-  )
   (wire (pts (xy 139.5476 96.6724) (xy 129.8956 96.6724))
     (stroke (width 0) (type default) (color 0 0 0 0))
   )
-  (wire (pts (xy 91.2876 91.5924) (xy 99.4156 91.5924))
+  (wire (pts (xy 91.2876 91.5924) (xy 95.0722 91.5924))
     (stroke (width 0) (type default) (color 0 0 0 0))
   )
@@
     (stroke (width 0) (type default) (color 0 0 0 0))
   )
+  (wire (pts (xy 97.0026 71.7804) (xy 132.8166 71.7804))
+    (stroke (width 0) (type default) (color 0 0 0 0))
+  )
+  (wire (pts (xy 95.0722 91.5924) (xy 99.4156 91.5924))
+    (stroke (width 0) (type default) (color 0 0 0 0))
+  )
+  (wire (pts (xy 97.0026 86.5124) (xy 97.0026 89.0524))
+    (stroke (width 0) (type default) (color 0 0 0 0))
+  )
   (wire (pts (xy 91.5416 106.8324) (xy 99.4156 106.8324))
     (stroke (width 0) (type default) (color 0 0 0 0))
@@
     (stroke (width 0) (type default) (color 0 0 0 0))
   )
-  (wire (pts (xy 97.0026 86.5124) (xy 97.0026 89.0524))
+  (wire (pts (xy 199.7964 74.4728) (xy 199.7964 83.8708))
+    (stroke (width 0) (type default) (color 0 0 0 0))
+  )
+  (wire (pts (xy 136.7028 91.5924) (xy 136.7028 77.5462))
+    (stroke (width 0) (type default) (color 0 0 0 0))
+  )
+  (wire (pts (xy 97.0026 71.7804) (xy 97.0026 86.5124))
+    (stroke (width 0) (type default) (color 0 0 0 0))
+  )
+  (wire (pts (xy 136.7028 77.5462) (xy 95.0722 77.5462))
     (stroke (width 0) (type default) (color 0 0 0 0))
   )
@@
     (stroke (width 0) (type default) (color 0 0 0 0))
   )
+  (wire (pts (xy 95.0722 77.5462) (xy 95.0722 91.5924))
+    (stroke (width 0) (type default) (color 0 0 0 0))
+  )
   (wire (pts (xy 139.5476 106.8324) (xy 129.8956 106.8324))
     (stroke (width 0) (type default) (color 0 0 0 0))
@@
     (stroke (width 0) (type default) (color 0 0 0 0))
   )
-  (wire (pts (xy 199.7964 83.8708) (xy 199.7964 78.1812))
+  (wire (pts (xy 132.8166 71.7804) (xy 132.8166 68.3514))
     (stroke (width 0) (type default) (color 0 0 0 0))
   )
@@
     (stroke (width 0) (type default) (color 0 0 0 0))
   )
+  (wire (pts (xy 176.3776 74.4728) (xy 199.7964 74.4728))
+    (stroke (width 0) (type default) (color 0 0 0 0))
+  )
   (wire (pts (xy 129.8956 86.5124) (xy 132.8166 86.5124))
     (stroke (width 0) (type default) (color 0 0 0 0))
@@
     (stroke (width 0) (type default) (color 0 0 0 0))
   )
-  (wire (pts (xy 91.2876 119.5324) (xy 99.4156 119.5324))
+  (wire (pts (xy 91.2876 119.5324) (xy 94.742 119.5324))
+    (stroke (width 0) (type default) (color 0 0 0 0))
+  )
+  (wire (pts (xy 94.742 125.349) (xy 132.0038 125.2982))
     (stroke (width 0) (type default) (color 0 0 0 0))
   )
@@
     (stroke (width 0) (type default) (color 0 0 0 0))
   )
-  (wire (pts (xy 132.8166 83.9724) (xy 132.8166 75.7174))
-    (stroke (width 0) (type default) (color 0 0 0 0))
-  )
-  (wire (pts (xy 132.8166 91.5924) (xy 132.8166 86.5124))
+  (wire (pts (xy 132.8166 83.9724) (xy 132.8166 71.7804))
     (stroke (width 0) (type default) (color 0 0 0 0))
   )
@@
     (stroke (width 0) (type default) (color 0 0 0 0))
   )
-  (wire (pts (xy 139.5476 119.5324) (xy 129.8956 119.5324))
+  (wire (pts (xy 176.3776 83.8708) (xy 176.3776 74.4728))
     (stroke (width 0) (type default) (color 0 0 0 0))
   )
@@
     (effects (font (size 1.27 1.27)) (justify right))
   )
-  (hierarchical_label "GND" (shape input) (at 97.0026 127.7874 270)
-    (effects (font (size 1.27 1.27)) (justify right))
-  )
   (hierarchical_label "+3.3V" (shape input) (at 139.5476 89.0524 0)
     (effects (font (size 1.27 1.27)) (justify left))
   )
-  (hierarchical_label "+3.3V" (shape input) (at 139.5476 119.5324 0)
-    (effects (font (size 1.27 1.27)) (justify left))
-  )
   (hierarchical_label "toMicroC_ADC_DB5" (shape input) (at 139.5476 106.8324 0)
     (effects (font (size 1.27 1.27)) (justify left))
@@
     (effects (font (size 1.27 1.27)) (justify left))
   )
-  (hierarchical_label "GND" (shape input) (at 199.7964 78.1812 90)
-    (effects (font (size 1.27 1.27)) (justify left))
-  )
   (hierarchical_label "toMicroC_ADC_DB0" (shape input) (at 91.5416 101.7524 180)
     (effects (font (size 1.27 1.27)) (justify right))
@@
     (effects (font (size 1.27 1.27)) (justify left))
   )
-  (hierarchical_label "GND" (shape input) (at 132.8166 75.7174 90)
-    (effects (font (size 1.27 1.27)) (justify left))
-  )
+  (hierarchical_label "GND" (shape input) (at 132.8166 68.3514 90)
+    (effects (font (size 1.27 1.27)) (justify left))
+  )

Commit message: V4 Ltspice
Parts:
- UB2: renamed from U4; footprint CEDCp:AD7606_M -> CEDCp_V2:AD7606_M
Changed lines of the file:
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@@
   (symbol (lib_id "CEDCp:AD7606_M") (at 101.9556 83.9724 0) (unit 1)
     (in_bom yes) (on_board yes) (fields_autoplaced)
-    (property "Reference" "U4" (id 0) (at 148.1328 73.8124 0))
-    (property "Value" "AD7606_M" (id 1) (at 148.1328 76.3524 0))
-    (property "Footprint" "CEDCp:AD7606_M" (id 2) (at 99.4156 83.9724 0)
+    (property "Reference" "UB2" (id 0) (at 148.1328 73.66 0))
+    (property "Value" "AD7606_M" (id 1) (at 148.1328 76.2 0))
+    (property "Footprint" "CEDCp_V2:AD7606_M" (id 2) (at 99.4156 83.9724 0)
       (effects (font (size 1.27 1.27)) hide)
     )
