File: Conversor_Digital_Analogico.kicad_sch (KiCad schematic)
At the start: 3 parts, among them U5 MCP4725

Commit message: Version V1 (Clearence + pads)
Parts:
- C13: value 1u -> 10u
Connections:
- net GND: now also U5.2 (VSS)
Changed lines of the file:
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@@
     (stroke (width 0) (type default) (color 0 0 0 0))
   )
-  (wire (pts (xy 152.4 119.38) (xy 152.4 121.92))
+  (wire (pts (xy 152.2476 118.11) (xy 152.2476 120.65))
     (stroke (width 0) (type default) (color 0 0 0 0))
   )
@@
     (effects (font (size 1.2954 1.2954) (thickness 0.2591) bold italic) (justify right))
   )
-  (hierarchical_label "GND" (shape input) (at 152.4 121.92 270)
+  (hierarchical_label "GND" (shape input) (at 152.2476 120.65 270)
     (effects (font (size 1.2954 1.2954) (thickness 0.2591) bold italic) (justify right))
   )
@@
       (effects (font (size 1.27 1.27)) (justify left))
     )
-    (property "Value" "1u" (id 1) (at 144.78 88.3284 0)
+    (property "Value" "10u" (id 1) (at 144.78 88.3284 0)
       (effects (font (size 1.27 1.27)) (justify left))
     )

Commit message: V4 Ltspice
Parts:
- removed U5: MCP4725, Connector_PinHeader_2.54mm:PinHeader_1x06_P2.54mm_Vertical, symbol CEDCp:MCP4725
- added U26: MCP4725_Placa, CEDCp_V2:MCP4725_Placa, symbol CEDCp_V2:MCP4725_Placa
- C7: renamed from C13; footprint CEDCp:Cap_1uF -> Capacitor_THT:CP_Radial_D4.0mm_P2.00mm
- renumbered C12 to C6
Connections:
- net +3.3V: now also U26.5 (VCC)
- net GND: now also U26.2 (GND), U26.6 (GND)
- net fromDAC_Vref: now also U26.1 (VOUT)
- net fromMicroC_DACI2C_SCL: now also U26.3 (SCL)
- net fromMicroC_DACI2C_SDA: now also U26.4 (SDA)
Changed lines of the file:
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@@
   (junction (at 137.16 92.71) (diameter 0) (color 0 0 0 0)
   )
+  (junction (at 142.24 81.28) (diameter 0) (color 0 0 0 0)
+  )
   (junction (at 130.81 81.28) (diameter 0) (color 0 0 0 0)
-  )
-  (junction (at 142.24 81.28) (diameter 0) (color 0 0 0 0)
   )
   (wire (pts (xy 130.81 92.71) (xy 130.81 91.44))
     (stroke (width 0) (type default) (color 0 0 0 0))
   )
-  (wire (pts (xy 143.8656 114.554) (xy 136.2456 114.554))
+  (wire (pts (xy 136.271 109.601) (xy 143.764 109.601))
     (stroke (width 0) (type default) (color 0 0 0 0))
   )
-  (wire (pts (xy 152.2476 105.41) (xy 152.2476 81.28))
-    (stroke (width 0) (type default) (color 0 0 0 0))
-  )
-  (wire (pts (xy 161.1376 111.76) (xy 173.99 111.76))
+  (wire (pts (xy 130.81 81.28) (xy 142.24 81.28))
     (stroke (width 0) (type default) (color 0 0 0 0))
   )
@@
     (stroke (width 0) (type default) (color 0 0 0 0))
   )
-  (wire (pts (xy 130.81 81.28) (xy 142.24 81.28))
-    (stroke (width 0) (type default) (color 0 0 0 0))
-  )
-  (wire (pts (xy 152.2476 118.11) (xy 152.2476 120.65))
-    (stroke (width 0) (type default) (color 0 0 0 0))
-  )
-  (wire (pts (xy 152.2476 81.28) (xy 142.24 81.28))
+  (wire (pts (xy 152.146 118.491) (xy 152.146 121.793))
     (stroke (width 0) (type default) (color 0 0 0 0))
   )
@@
     (stroke (width 0) (type default) (color 0 0 0 0))
   )
+  (wire (pts (xy 136.271 114.935) (xy 143.764 114.935))
+    (stroke (width 0) (type default) (color 0 0 0 0))
+  )
   (wire (pts (xy 127 81.28) (xy 130.81 81.28))
+    (stroke (width 0) (type default) (color 0 0 0 0))
+  )
+  (wire (pts (xy 161.036 112.141) (xy 163.957 112.141))
+    (stroke (width 0) (type default) (color 0 0 0 0))
+  )
+  (wire (pts (xy 142.24 81.28) (xy 152.146 81.28))
+    (stroke (width 0) (type default) (color 0 0 0 0))
+  )
+  (wire (pts (xy 136.271 112.141) (xy 143.764 112.141))
+    (stroke (width 0) (type default) (color 0 0 0 0))
+  )
+  (wire (pts (xy 152.146 81.28) (xy 152.146 105.791))
     (stroke (width 0) (type default) (color 0 0 0 0))
   )
@@
     (stroke (width 0) (type default) (color 0 0 0 0))
   )
-  (wire (pts (xy 136.2456 109.22) (xy 143.8656 109.22))
-    (stroke (width 0) (type default) (color 0 0 0 0))
-  )
-  (wire (pts (xy 143.8656 111.76) (xy 136.2456 111.76))
-    (stroke (width 0) (type default) (color 0 0 0 0))
-  )
   (text "A0= debera conectarse a masa o 3.3V segun la direccion\n I2C que se le asisgne al DAC en el bus de comunicacion I2C"
     (at 64.516 131.699 0)
@@
   )
   (text "C6 y C7 se deben conectar lo mas cercano posible \nal pin Vdd del DAC para filtrar ruidos de la \nalimentacion que afectan la performance del DAC\nC6: Capacitor Ceramico\nC7: Capacitor Tantalio"
-    (at 57.277 92.964 0)
+    (at 158.8262 91.059 0)
     (effects (font (size 1.27 1.27) (thickness 0.254) bold) (justify left bottom))
   )
@@
     (effects (font (size 3.5 3.5) (thickness 0.5994) bold) (justify left bottom))
   )
-  (hierarchical_label "fromMicroC_DACI2C_SDA" (shape input) (at 136.2456 109.22 180)
+  (hierarchical_label "fromMicroC_DACI2C_SDA" (shape input) (at 136.271 109.601 180)
     (effects (font (size 1.2954 1.2954) (thickness 0.2591) bold italic) (justify right))
   )
-  (hierarchical_label "fromDAC_Vref" (shape output) (at 173.99 111.76 0)
+  (hierarchical_label "fromDAC_Vref" (shape output) (at 163.957 112.141 0)
     (effects (font (size 1.2954 1.2954) (thickness 0.2591) bold italic) (justify left))
   )
@@
     (effects (font (size 1.2954 1.2954) (thickness 0.2591) bold italic) (justify right))
   )
-  (hierarchical_label "GND" (shape input) (at 152.2476 120.65 270)
+  (hierarchical_label "GND" (shape input) (at 152.146 121.793 270)
     (effects (font (size 1.2954 1.2954) (thickness 0.2591) bold italic) (justify right))
   )
-  (hierarchical_label "GND" (shape input) (at 136.2456 114.554 180)
+  (hierarchical_label "GND" (shape input) (at 136.271 114.935 180)
     (effects (font (size 1.2954 1.2954) (thickness 0.2591) bold italic) (justify right))
   )
@@
     (effects (font (size 1.2954 1.2954) (thickness 0.2591) bold italic) (justify right))
   )
-  (hierarchical_label "fromMicroC_DACI2C_SCL" (shape input) (at 136.2456 111.76 180)
+  (hierarchical_label "fromMicroC_DACI2C_SCL" (shape input) (at 136.271 112.141 180)
     (effects (font (size 1.2954 1.2954) (thickness 0.2591) bold italic) (justify right))
   )
   (symbol (lib_id "Capacitor_2:C315C222K1R5CA") (at 130.81 83.82 270) (unit 1)
     (in_bom yes) (on_board yes)
-    (property "Reference" "C12" (id 0) (at 135.89 85.09 90))
+    (property "Reference" "C6" (id 0) (at 135.89 85.09 90))
     (property "Value" "0.1u" (id 1) (at 135.89 87.63 90))
     (property "Footprint" "Capacitor_THT:C_Disc_D7.5mm_W2.5mm_P5.00mm" (id 2) (at 121.666 87.63 0)
@@
     (pin "2")
   )
-  (symbol (lib_id "CEDCp:MCP4725") (at 152.2476 111.76 0) (unit 1)
+  (symbol (lib_id "Device:C_Polarized_Small") (at 142.24 87.6046 0) (unit 1)
     (in_bom yes) (on_board yes) (fields_autoplaced)
-    (property "Reference" "U5" (id 0) (at 165.1 107.2808 0))
-    (property "Value" "MCP4725" (id 1) (at 165.1 109.8208 0))
-    (property "Footprint" "Connector_PinHeader_2.54mm:PinHeader_1x06_P2.54mm_Vertical" (id 2) (at 158.3436 104.902 0)
+    (property "Reference" "C7" (id 0) (at 144.78 85.7884 0)
+      (effects (font (size 1.27 1.27)) (justify left))
+    )
+    (property "Value" "10u" (id 1) (at 144.78 88.3284 0)
+      (effects (font (size 1.27 1.27)) (justify left))
+    )
+    (property "Footprint" "Capacitor_THT:CP_Radial_D4.0mm_P2.00mm" (id 2) (at 142.24 87.6046 0)
       (effects (font (size 1.27 1.27)) hide)
     )
-    (property "Datasheet" "" (id 3) (at 158.3436 104.902 0)
+    (property "Datasheet" "~" (id 3) (at 142.24 87.6046 0)
+      (effects (font (size 1.27 1.27)) hide)
+    )
+    (pin "1")
+    (pin "2")
+  )
+  (symbol (lib_id "CEDCp_V2:MCP4725_Placa") (at 152.146 112.141 0) (unit 1)
+    (in_bom yes) (on_board yes) (fields_autoplaced)
+    (property "Reference" "U26" (id 0) (at 167.64 107.6618 0))
+    (property "Value" "MCP4725_Placa" (id 1) (at 167.64 110.2018 0))
+    (property "Footprint" "CEDCp_V2:MCP4725_Placa" (id 2) (at 158.242 105.283 0)
+      (effects (font (size 1.27 1.27)) hide)
+    )
+    (property "Datasheet" "" (id 3) (at 158.242 105.283 0)
       (effects (font (size 1.27 1.27)) hide)
     )
@@
     (pin "6")
   )
-  (symbol (lib_id "Device:C_Polarized_Small") (at 142.24 87.6046 0) (unit 1)
-    (in_bom yes) (on_board yes) (fields_autoplaced)
-    (property "Reference" "C13" (id 0) (at 144.78 85.7884 0)
-      (effects (font (size 1.27 1.27)) (justify left))
-    )
-    (property "Value" "10u" (id 1) (at 144.78 88.3284 0)
-      (effects (font (size 1.27 1.27)) (justify left))
-    )
-    (property "Footprint" "CEDCp:Cap_1uF" (id 2) (at 142.24 87.6046 0)
-      (effects (font (size 1.27 1.27)) hide)
-    )
-    (property "Datasheet" "~" (id 3) (at 142.24 87.6046 0)
-      (effects (font (size 1.27 1.27)) hide)
-    )
-    (pin "1")
-    (pin "2")
-  )
 )
