File: Lazo Realimentacion de Corriente (Lazo 1).kicad_sch (KiCad schematic)
At the start: 15 parts, among them U6 OPA604

Commit message: V4 Ltspice
Parts:
- R11: renamed from R20; footprint CEDCp:Resistencia_0,25W -> CEDCp_V2:Resistencia_0,25W
- R16: renamed from R21; footprint CEDCp:Resistencia_0,25W -> CEDCp_V2:Resistencia_0,25W
- R17: renamed from R22; footprint CEDCp:Resistencia_0,25W -> CEDCp_V2:Resistencia_0,25W
- R21: renamed from R18; footprint CEDCp:Resistencia_0,25W -> CEDCp_V2:Resistencia_0,25W
- R23: footprint CEDCp:Resistencia_0,25W -> CEDCp_V2:Resistencia_0,25W
- R24: renamed from R15; footprint CEDCp:Resistencia_0,25W -> CEDCp_V2:Resistencia_0,25W
- R25: renamed from R16; footprint CEDCp:Resistencia_0,25W -> CEDCp_V2:Resistencia_0,25W
- R26: renamed from R24; footprint CEDCp:Resistencia_0,25W -> CEDCp_V2:Resistencia_0,25W
- R27: renamed from R17; footprint CEDCp:Resistencia_0,25W -> CEDCp_V2:Resistencia_0,25W
- R8: renamed from R19; footprint CEDCp:Resistencia_0,25W -> CEDCp_V2:Resistencia_0,25W
- renumbered C5 to C1, C4 to C5, U6 to U11
Connections:
- net Error1: now also U11.6 (Out)
Other:
- note added: "Resistencias de offset 250k en vez de 100k Capacitores de desacople.."
Changed lines of the file:
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@@
   (junction (at 163.83 104.14) (diameter 0) (color 0 0 0 0)
   )
+  (junction (at 163.83 111.76) (diameter 0) (color 0 0 0 0)
+  )
+  (junction (at 163.83 119.38) (diameter 0) (color 0 0 0 0)
+  )
   (junction (at 198.247 93.98) (diameter 0) (color 0 0 0 0)
-  )
-  (junction (at 163.83 111.76) (diameter 0) (color 0 0 0 0)
-  )
-  (junction (at 198.2216 93.98) (diameter 0) (color 0 0 0 0)
-  )
-  (junction (at 163.83 119.38) (diameter 0) (color 0 0 0 0)
   )
   (junction (at 180.721 101.6) (diameter 0) (color 0 0 0 0)
@@
     (stroke (width 0) (type default) (color 0 0 0 0))
   )
-  (wire (pts (xy 190.2968 93.98) (xy 198.2216 93.98))
-    (stroke (width 0) (type default) (color 0 0 0 0))
-  )
   (wire (pts (xy 132.588 78.74) (xy 132.588 82.931))
     (stroke (width 0) (type default) (color 0 0 0 0))
@@
     (stroke (width 0) (type default) (color 0 0 0 0))
   )
+  (wire (pts (xy 190.2968 93.98) (xy 198.247 93.98))
+    (stroke (width 0) (type default) (color 0 0 0 0))
+  )
+  (wire (pts (xy 182.626 99.187) (xy 182.626 109.0422))
+    (stroke (width 0) (type default) (color 0 0 0 0))
+  )
+  (wire (pts (xy 180.975 69.85) (xy 187.96 69.85))
+    (stroke (width 0) (type default) (color 0 0 0 0))
+  )
+  (wire (pts (xy 157.48 104.14) (xy 163.83 104.14))
+    (stroke (width 0) (type default) (color 0 0 0 0))
+  )
+  (wire (pts (xy 163.83 127) (xy 163.83 130.81))
+    (stroke (width 0) (type default) (color 0 0 0 0))
+  )
   (wire (pts (xy 198.247 93.98) (xy 212.09 93.98))
-    (stroke (width 0) (type default) (color 0 0 0 0))
-  )
-  (wire (pts (xy 182.626 99.187) (xy 182.626 109.0422))
-    (stroke (width 0) (type default) (color 0 0 0 0))
-  )
-  (wire (pts (xy 180.975 69.85) (xy 187.96 69.85))
-    (stroke (width 0) (type default) (color 0 0 0 0))
-  )
-  (wire (pts (xy 157.48 104.14) (xy 163.83 104.14))
-    (stroke (width 0) (type default) (color 0 0 0 0))
-  )
-  (wire (pts (xy 163.83 127) (xy 163.83 130.81))
     (stroke (width 0) (type default) (color 0 0 0 0))
   )
@@
   (text "C3 capacitor ceramico" (at 170.18 138.43 0)
     (effects (font (size 1.4986 1.4986) (thickness 0.2997) bold) (justify left bottom))
+  )
+  (text "Resistencias de offset 250k en vez de 100k\nCapacitores de desacople.."
+    (at 228.1682 80.4164 0)
+    (effects (font (size 3 3) bold italic) (justify left bottom))
   )
   (text "Lazo Realimentacion de Corriente (Lazo 1)" (at 34.798 36.957 0)
@@
   (symbol (lib_id "Capacitor_2:C315C222K1R5CA") (at 176.911 101.6 270) (unit 1)
     (in_bom yes) (on_board yes)
-    (property "Reference" "C4" (id 0) (at 173.101 102.87 90)
+    (property "Reference" "C5" (id 0) (at 173.101 102.87 90)
       (effects (font (size 1.524 1.524)))
     )
@@
   (symbol (lib_id "Capacitor_2:C315C222K1R5CA") (at 185.039 78.5368 270) (unit 1)
     (in_bom yes) (on_board yes)
-    (property "Reference" "C5" (id 0) (at 190.119 79.8068 90)
+    (property "Reference" "C1" (id 0) (at 190.119 79.8068 90)
       (effects (font (size 1.524 1.524)))
     )
@@
   (symbol (lib_id "Device:R_Small") (at 132.588 85.471 0) (unit 1)
     (in_bom yes) (on_board yes)
-    (property "Reference" "R15" (id 0) (at 133.35 85.471 0)
+    (property "Reference" "R24" (id 0) (at 133.35 85.471 0)
       (effects (font (size 1.27 1.27)) (justify left))
     )
@@
       (effects (font (size 1 1)) (justify left))
     )
-    (property "Footprint" "CEDCp:Resistencia_0,25W" (id 2) (at 132.588 85.471 0)
+    (property "Footprint" "CEDCp_V2:Resistencia_0,25W" (id 2) (at 132.588 85.471 0)
       (effects (font (size 1.27 1.27)) hide)
     )
@@
   (symbol (lib_id "Device:R_Small") (at 154.94 104.14 90) (unit 1)
     (in_bom yes) (on_board yes)
-    (property "Reference" "R19" (id 0) (at 156.464 102.489 90)
+    (property "Reference" "R8" (id 0) (at 156.464 102.489 90)
       (effects (font (size 1.27 1.27)) (justify left))
     )
@@
       (effects (font (size 1 1)) (justify left))
     )
-    (property "Footprint" "CEDCp:Resistencia_0,25W" (id 2) (at 154.94 104.14 0)
+    (property "Footprint" "CEDCp_V2:Resistencia_0,25W" (id 2) (at 154.94 104.14 0)
       (effects (font (size 1.27 1.27)) hide)
     )
@@
   (symbol (lib_id "CEDCp:OPA604") (at 181.61 93.472 0) (unit 1)
     (in_bom yes) (on_board yes) (fields_autoplaced)
-    (property "Reference" "U6" (id 0) (at 192.8622 89.281 0))
-    (property "Value" "OPA604" (id 1) (at 192.8622 91.821 0))
+    (property "Reference" "U11" (id 0) (at 193.04 89.281 0))
+    (property "Value" "OPA604" (id 1) (at 193.04 91.821 0))
     (property "Footprint" "CEDCp:OPA604" (id 2) (at 182.0672 81.534 0)
       (effects (font (size 1.27 1.27)) hide)
@@
   (symbol (lib_id "Device:R_Small") (at 154.94 111.76 90) (unit 1)
     (in_bom yes) (on_board yes)
-    (property "Reference" "R20" (id 0) (at 156.464 110.109 90)
+    (property "Reference" "R11" (id 0) (at 156.464 110.109 90)
       (effects (font (size 1.27 1.27)) (justify left))
     )
@@
       (effects (font (size 1 1)) (justify left))
     )
-    (property "Footprint" "CEDCp:Resistencia_0,25W" (id 2) (at 154.94 111.76 0)
+    (property "Footprint" "CEDCp_V2:Resistencia_0,25W" (id 2) (at 154.94 111.76 0)
       (effects (font (size 1.27 1.27)) hide)
     )
@@
   (symbol (lib_id "Device:R_Small") (at 152.4 91.44 90) (unit 1)
     (in_bom yes) (on_board yes)
-    (property "Reference" "R18" (id 0) (at 153.924 89.789 90)
+    (property "Reference" "R21" (id 0) (at 153.924 89.789 90)
       (effects (font (size 1.27 1.27)) (justify left))
     )
@@
       (effects (font (size 1 1)) (justify left))
     )
-    (property "Footprint" "CEDCp:Resistencia_0,25W" (id 2) (at 152.4 91.44 0)
+    (property "Footprint" "CEDCp_V2:Resistencia_0,25W" (id 2) (at 152.4 91.44 0)
       (effects (font (size 1.27 1.27)) hide)
     )
@@
   (symbol (lib_id "Device:R_Small") (at 132.588 104.775 0) (unit 1)
     (in_bom yes) (on_board yes)
-    (property "Reference" "R17" (id 0) (at 133.35 104.775 0)
+    (property "Reference" "R27" (id 0) (at 133.35 104.775 0)
       (effects (font (size 1.27 1.27)) (justify left))
     )
@@
       (effects (font (size 1 1)) (justify left))
     )
-    (property "Footprint" "CEDCp:Resistencia_0,25W" (id 2) (at 132.588 104.775 0)
+    (property "Footprint" "CEDCp_V2:Resistencia_0,25W" (id 2) (at 132.588 104.775 0)
       (effects (font (size 1.27 1.27)) hide)
     )
@@
       (effects (font (size 1 1)) (justify left))
     )
-    (property "Footprint" "CEDCp:Resistencia_0,25W" (id 2) (at 178.435 69.85 0)
+    (property "Footprint" "CEDCp_V2:Resistencia_0,25W" (id 2) (at 178.435 69.85 0)
       (effects (font (size 1.27 1.27)) hide)
     )
@@
   (symbol (lib_id "Device:R_Small") (at 154.94 119.38 90) (unit 1)
     (in_bom yes) (on_board yes)
-    (property "Reference" "R21" (id 0) (at 156.464 117.729 90)
+    (property "Reference" "R16" (id 0) (at 156.464 117.729 90)
       (effects (font (size 1.27 1.27)) (justify left))
     )
@@
       (effects (font (size 1 1)) (justify left))
     )
-    (property "Footprint" "CEDCp:Resistencia_0,25W" (id 2) (at 154.94 119.38 0)
+    (property "Footprint" "CEDCp_V2:Resistencia_0,25W" (id 2) (at 154.94 119.38 0)
       (effects (font (size 1.27 1.27)) hide)
     )
@@
   (symbol (lib_id "Device:R_Small") (at 154.94 127 90) (unit 1)
     (in_bom yes) (on_board yes)
-    (property "Reference" "R22" (id 0) (at 156.464 125.349 90)
+    (property "Reference" "R17" (id 0) (at 156.464 125.349 90)
       (effects (font (size 1.27 1.27)) (justify left))
     )
@@
       (effects (font (size 1 1)) (justify left))
     )
-    (property "Footprint" "CEDCp:Resistencia_0,25W" (id 2) (at 154.94 127 0)
+    (property "Footprint" "CEDCp_V2:Resistencia_0,25W" (id 2) (at 154.94 127 0)
       (effects (font (size 1.27 1.27)) hide)
     )
@@
   (symbol (lib_id "Device:R_Small") (at 132.588 96.52 0) (unit 1)
     (in_bom yes) (on_board yes)
-    (property "Reference" "R16" (id 0) (at 133.35 96.52 0)
+    (property "Reference" "R25" (id 0) (at 133.35 96.52 0)
       (effects (font (size 1.27 1.27)) (justify left))
     )
@@
       (effects (font (size 1 1)) (justify left))
     )
-    (property "Footprint" "CEDCp:Resistencia_0,25W" (id 2) (at 132.588 96.52 0)
+    (property "Footprint" "CEDCp_V2:Resistencia_0,25W" (id 2) (at 132.588 96.52 0)
       (effects (font (size 1.27 1.27)) hide)
     )
@@
   (symbol (lib_id "Device:R_Small") (at 190.5 69.85 90) (unit 1)
     (in_bom yes) (on_board yes)
-    (property "Reference" "R24" (id 0) (at 192.024 68.199 90)
+    (property "Reference" "R26" (id 0) (at 192.024 68.199 90)
       (effects (font (size 1.27 1.27)) (justify left))
     )
@@
       (effects (font (size 1 1)) (justify left))
     )
-    (property "Footprint" "CEDCp:Resistencia_0,25W" (id 2) (at 190.5 69.85 0)
-      (effects (font (size 1.27 1.27)) hide)
-    )
+    (property "Footprint" "CEDCp_V2:Resistencia_0,25W" (id 2) (at 190.5 69.85 0)
+      (effects (font (size 1.27 1.27)) hide)
+    )
