File: Lazo Realimentacion de Voltaje (Lazo 2).kicad_sch (KiCad schematic)
At the start: 14 parts, among them U7 OPA604

Commit message: Pads mas grandes y correccion de vias
Other:
- note added: "U9 es un preset multivueltas usado para ajustar de forma precisa el voltaje de 1.1V requeridos."
- note removed: "U9 es un preset multivueltas usado para ajustar de forma precisa el voltaje de 1.1V requeridos. El valor de R19 ya considera la posibilidad de que el preset quede con una resitencia de 0 al manipularse por tanto limita la corriente a valores adecuados"
Changed lines of the file:
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@@
     (stroke (width 0) (type default) (color 0 0 0 0))
   )
-  (text "U9 es un preset multivueltas usado para\najustar de forma precisa el voltaje de 1.1V requeridos.\nEl valor de R19 ya considera la posibilidad de que el \npreset quede con una resitencia de 0 al manipularse \npor tanto limita la corriente a valores adecuados"
+  (text "U9 es un preset multivueltas usado para\najustar de forma precisa el voltaje de 1.1V requeridos."
     (at 195.58 158.115 0)
     (effects (font (size 1.4986 1.4986) (thickness 0.2997) bold) (justify left bottom))

Commit message: V4 Ltspice
Parts:
- R13: renamed from R29; footprint CEDCp:Resistencia_0,25W -> CEDCp_V2:Resistencia_0,25W
- R15: renamed from R30; footprint CEDCp:Resistencia_0,25W -> CEDCp_V2:Resistencia_0,25W
- R18: renamed from R28; footprint CEDCp:Resistencia_0,25W -> CEDCp_V2:Resistencia_0,25W
- R38: renamed from R25; footprint CEDCp:Resistencia_0,25W -> CEDCp_V2:Resistencia_0,25W
- R39: renamed from R26; footprint CEDCp:Resistencia_0,25W -> CEDCp_V2:Resistencia_0,25W
- R43: renamed from R27; footprint CEDCp:Resistencia_0,25W -> CEDCp_V2:Resistencia_0,25W
- renumbered C14 to C11, C15 to C9, D2 to D8, U7 to U5
Other:
- note added: "Resistencias de offset 250k en vez de 100k Capacitores de desacople.."
Changed lines of the file:
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@@
     (effects (font (size 1.4986 1.4986) (thickness 0.2997) bold) (justify left bottom))
+  )
+  (text "Resistencias de offset 250k en vez de 100k\nCapacitores de desacople.."
+    (at 204.8256 97.6122 0)
+    (effects (font (size 3 3) bold italic) (justify left bottom))
   )
   (text "U21 y U22 son un presets\nmultivueltas" (at 39.751 111.379 0)
@@
   (symbol (lib_id "Diode:BZX384-xxx") (at 108.077 116.84 270) (unit 1)
     (in_bom yes) (on_board yes)
-    (property "Reference" "D2" (id 0) (at 109.728 116.967 90)
+    (property "Reference" "D8" (id 0) (at 109.728 116.967 90)
       (effects (font (size 1.27 1.27)) (justify left))
     )
@@
   (symbol (lib_id "Capacitor_2:C315C222K1R5CA") (at 170.053 127 90) (unit 1)
     (in_bom yes) (on_board yes)
-    (property "Reference" "C14" (id 0) (at 164.973 120.65 90)
+    (property "Reference" "C11" (id 0) (at 164.973 120.65 90)
       (effects (font (size 1.524 1.524)))
     )
@@
   (symbol (lib_id "Capacitor_2:C315C222K1R5CA") (at 178.181 96.3422 270) (unit 1)
     (in_bom yes) (on_board yes)
-    (property "Reference" "C15" (id 0) (at 183.261 97.6122 90)
+    (property "Reference" "C9" (id 0) (at 183.261 97.6122 90)
       (effects (font (size 1.524 1.524)))
     )
@@
   (symbol (lib_id "Device:R_Small") (at 90.297 88.138 0) (unit 1)
     (in_bom yes) (on_board yes)
-    (property "Reference" "R26" (id 0) (at 91.186 88.265 0)
+    (property "Reference" "R39" (id 0) (at 91.186 88.265 0)
       (effects (font (size 1.27 1.27)) (justify left))
     )
@@
       (effects (font (size 1 1)) (justify left))
     )
-    (property "Footprint" "CEDCp:Resistencia_0,25W" (id 2) (at 90.297 88.138 0)
+    (property "Footprint" "CEDCp_V2:Resistencia_0,25W" (id 2) (at 90.297 88.138 0)
       (effects (font (size 1.27 1.27)) hide)
     )
@@
   (symbol (lib_id "Device:R_Small") (at 174.625 88.773 90) (unit 1)
     (in_bom yes) (on_board yes)
-    (property "Reference" "R30" (id 0) (at 175.895 87.122 90)
+    (property "Reference" "R15" (id 0) (at 175.895 87.122 90)
       (effects (font (size 1.27 1.27)) (justify left))
     )
@@
       (effects (font (size 0.9 0.9)) (justify left))
     )
-    (property "Footprint" "CEDCp:Resistencia_0,25W" (id 2) (at 174.625 88.773 0)
+    (property "Footprint" "CEDCp_V2:Resistencia_0,25W" (id 2) (at 174.625 88.773 0)
       (effects (font (size 1.27 1.27)) hide)
     )
@@
   (symbol (lib_id "Device:R_Small") (at 146.05 116.84 90) (unit 1)
     (in_bom yes) (on_board yes)
-    (property "Reference" "R29" (id 0) (at 147.32 115.189 90)
+    (property "Reference" "R13" (id 0) (at 147.32 115.189 90)
       (effects (font (size 1.27 1.27)) (justify left))
     )
@@
       (effects (font (size 0.9 0.9)) (justify left))
     )
-    (property "Footprint" "CEDCp:Resistencia_0,25W" (id 2) (at 146.05 116.84 0)
+    (property "Footprint" "CEDCp_V2:Resistencia_0,25W" (id 2) (at 146.05 116.84 0)
       (effects (font (size 1.27 1.27)) hide)
     )
@@
   (symbol (lib_id "Device:R_Small") (at 90.297 119.888 0) (unit 1)
     (in_bom yes) (on_board yes)
-    (property "Reference" "R27" (id 0) (at 91.313 119.888 0)
+    (property "Reference" "R43" (id 0) (at 91.313 119.888 0)
       (effects (font (size 1.27 1.27)) (justify left))
     )
@@
       (effects (font (size 1 1)) (justify left))
     )
-    (property "Footprint" "CEDCp:Resistencia_0,25W" (id 2) (at 90.297 119.888 0)
+    (property "Footprint" "CEDCp_V2:Resistencia_0,25W" (id 2) (at 90.297 119.888 0)
       (effects (font (size 1.27 1.27)) hide)
     )
@@
   (symbol (lib_id "CEDCp:OPA604") (at 174.752 111.252 0) (unit 1)
     (in_bom yes) (on_board yes) (fields_autoplaced)
-    (property "Reference" "U7" (id 0) (at 186.0042 107.061 0))
-    (property "Value" "OPA604" (id 1) (at 186.0042 109.601 0))
+    (property "Reference" "U5" (id 0) (at 185.42 107.061 0))
+    (property "Value" "OPA604" (id 1) (at 185.42 109.601 0))
     (property "Footprint" "CEDCp:OPA604" (id 2) (at 175.2092 99.314 0)
       (effects (font (size 1.27 1.27)) hide)
@@
   (symbol (lib_id "Device:R_Small") (at 146.05 109.22 90) (unit 1)
     (in_bom yes) (on_board yes)
-    (property "Reference" "R28" (id 0) (at 147.32 107.569 90)
+    (property "Reference" "R18" (id 0) (at 147.32 107.569 90)
       (effects (font (size 1.27 1.27)) (justify left))
     )
@@
       (effects (font (size 0.9 0.9)) (justify left))
     )
-    (property "Footprint" "CEDCp:Resistencia_0,25W" (id 2) (at 146.05 109.22 0)
+    (property "Footprint" "CEDCp_V2:Resistencia_0,25W" (id 2) (at 146.05 109.22 0)
       (effects (font (size 1.27 1.27)) hide)
     )
@@
   (symbol (lib_id "Device:R_Small") (at 90.297 79.248 0) (unit 1)
     (in_bom yes) (on_board yes)
-    (property "Reference" "R25" (id 0) (at 91.186 79.375 0)
+    (property "Reference" "R38" (id 0) (at 91.186 79.375 0)
       (effects (font (size 1.27 1.27)) (justify left))
     )
@@
       (effects (font (size 1 1)) (justify left))
     )
-    (property "Footprint" "CEDCp:Resistencia_0,25W" (id 2) (at 90.297 79.248 0)
-      (effects (font (size 1.27 1.27)) hide)
-    )
+    (property "Footprint" "CEDCp_V2:Resistencia_0,25W" (id 2) (at 90.297 79.248 0)
+      (effects (font (size 1.27 1.27)) hide)
+    )
