File: Medicion Corriente Total en la CEP (ADC).kicad_sch (KiCad schematic)
At the start: 11 parts, among them U8 OPA604

Commit message: V4 Ltspice
Parts:
- R29: renamed from R31; footprint CEDCp:Resistencia_0,25W -> CEDCp_V2:Resistencia_0,25W
- R31: renamed from R32; footprint CEDCp:Resistencia_0,25W -> CEDCp_V2:Resistencia_0,25W
- R34: renamed from R33; footprint CEDCp:Resistencia_0,25W -> CEDCp_V2:Resistencia_0,25W
- R35: renamed from R34; footprint CEDCp:Resistencia_0,25W -> CEDCp_V2:Resistencia_0,25W
- R36: renamed from R35; footprint CEDCp:Resistencia_0,25W -> CEDCp_V2:Resistencia_0,25W
- R37: renamed from R36; footprint CEDCp:Resistencia_0,25W -> CEDCp_V2:Resistencia_0,25W
- R41: renamed from R38; footprint CEDCp:Resistencia_0,25W -> CEDCp_V2:Resistencia_0,25W
- renumbered C2 to C13, C1 to C15, RV8 to U11, U8 to U20
Other:
- note added: "DUDA: ¿Que valor es el de los capacitores de desacople? 0.1u o 1u (No se corresponden) El valor del potenciometro de ajuste es de: 250k (No se corresponde con el LTSPICE)"
Changed lines of the file:
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@@
     (effects (font (size 1.4986 1.4986) (thickness 0.2997) bold) (justify left bottom))
+  )
+  (text "DUDA: \n¿Que valor es el de los capacitores de desacople?\n    0.1u o 1u (No se corresponden)\nEl valor del potenciometro de ajuste es de:\n250k (No se corresponde con el LTSPICE)\n\n"
+    (at 178.1302 80.0354 0)
+    (effects (font (size 3 3) (thickness 0.6) bold italic) (justify left bottom))
   )
   (text "R36, R37 y R41 al 1%" (at 83.439 93.091 0)
@@
   (symbol (lib_id "Capacitor_2:C315C222K1R5CA") (at 146.6342 103.886 270) (unit 1)
     (in_bom yes) (on_board yes)
-    (property "Reference" "C1" (id 0) (at 141.5542 105.156 90)
+    (property "Reference" "C15" (id 0) (at 141.5542 105.156 90)
       (effects (font (size 1.524 1.524)))
     )
@@
   (symbol (lib_id "Device:R_Small") (at 130.8862 98.044 90) (unit 1)
     (in_bom yes) (on_board yes)
-    (property "Reference" "R31" (id 0) (at 132.1562 96.139 90)
+    (property "Reference" "R29" (id 0) (at 132.1562 96.139 90)
       (effects (font (size 1.27 1.27)) (justify left))
     )
@@
       (effects (font (size 1 1)) (justify left))
     )
-    (property "Footprint" "CEDCp:Resistencia_0,25W" (id 2) (at 130.8862 98.044 0)
+    (property "Footprint" "CEDCp_V2:Resistencia_0,25W" (id 2) (at 130.8862 98.044 0)
       (effects (font (size 1.27 1.27)) hide)
     )
@@
   (symbol (lib_id "Capacitor_2:C315C222K1R5CA") (at 154.7622 77.978 270) (unit 1)
     (in_bom yes) (on_board yes)
-    (property "Reference" "C2" (id 0) (at 159.8422 79.248 90)
+    (property "Reference" "C13" (id 0) (at 159.8422 79.248 90)
       (effects (font (size 1.524 1.524)))
     )
@@
   (symbol (lib_id "Device:R_Small") (at 150.0124 71.374 90) (unit 1)
     (in_bom yes) (on_board yes)
-    (property "Reference" "R36" (id 0) (at 151.2824 69.469 90)
+    (property "Reference" "R37" (id 0) (at 151.2824 69.469 90)
       (effects (font (size 1.27 1.27)) (justify left))
     )
@@
       (effects (font (size 1 1)) (justify left))
     )
-    (property "Footprint" "CEDCp:Resistencia_0,25W" (id 2) (at 150.0124 71.374 0)
+    (property "Footprint" "CEDCp_V2:Resistencia_0,25W" (id 2) (at 150.0124 71.374 0)
       (effects (font (size 1.27 1.27)) hide)
     )
@@
   (symbol (lib_id "Device:R_Small") (at 160.8074 71.374 90) (unit 1)
     (in_bom yes) (on_board yes)
-    (property "Reference" "R38" (id 0) (at 162.0774 69.469 90)
+    (property "Reference" "R41" (id 0) (at 162.0774 69.469 90)
       (effects (font (size 1.27 1.27)) (justify left))
     )
@@
       (effects (font (size 1 1)) (justify left))
     )
-    (property "Footprint" "CEDCp:Resistencia_0,25W" (id 2) (at 160.8074 71.374 0)
+    (property "Footprint" "CEDCp_V2:Resistencia_0,25W" (id 2) (at 160.8074 71.374 0)
       (effects (font (size 1.27 1.27)) hide)
     )
@@
   (symbol (lib_id "Device:R_Small") (at 136.0424 81.534 90) (unit 1)
     (in_bom yes) (on_board yes)
-    (property "Reference" "R35" (id 0) (at 137.3124 79.629 90)
+    (property "Reference" "R36" (id 0) (at 137.3124 79.629 90)
       (effects (font (size 1.27 1.27)) (justify left))
     )
@@
       (effects (font (size 1 1)) (justify left))
     )
-    (property "Footprint" "CEDCp:Resistencia_0,25W" (id 2) (at 136.0424 81.534 0)
+    (property "Footprint" "CEDCp_V2:Resistencia_0,25W" (id 2) (at 136.0424 81.534 0)
       (effects (font (size 1.27 1.27)) hide)
     )
@@
     (pin "2")
   )
-  (symbol (lib_name "OPA604_1") (lib_id "CEDCp:OPA604") (at 151.3332 94.996 0) (unit 1)
-    (in_bom yes) (on_board yes)
-    (property "Reference" "U8" (id 0) (at 148.0566 88.8492 0))
+  (symbol (lib_id "CEDCp:OPA604") (at 151.3332 94.996 0) (unit 1)
+    (in_bom yes) (on_board yes)
+    (property "Reference" "U20" (id 0) (at 148.0566 88.8492 0))
     (property "Value" "OPA604" (id 1) (at 159.4866 98.2472 0))
     (property "Footprint" "CEDCp:OPA604" (id 2) (at 151.7904 83.058 0)
@@
   (symbol (lib_id "Device:R_Small") (at 130.8862 105.664 90) (unit 1)
     (in_bom yes) (on_board yes)
-    (property "Reference" "R32" (id 0) (at 132.1562 103.759 90)
+    (property "Reference" "R31" (id 0) (at 132.1562 103.759 90)
       (effects (font (size 1.27 1.27)) (justify left))
     )
@@
       (effects (font (size 1 1)) (justify left))
     )
-    (property "Footprint" "CEDCp:Resistencia_0,25W" (id 2) (at 130.8862 105.664 0)
+    (property "Footprint" "CEDCp_V2:Resistencia_0,25W" (id 2) (at 130.8862 105.664 0)
       (effects (font (size 1.27 1.27)) hide)
     )
@@
   (symbol (lib_id "Device:R_Small") (at 130.8862 113.284 90) (unit 1)
     (in_bom yes) (on_board yes)
-    (property "Reference" "R33" (id 0) (at 132.1562 111.379 90)
+    (property "Reference" "R34" (id 0) (at 132.1562 111.379 90)
       (effects (font (size 1.27 1.27)) (justify left))
     )
@@
       (effects (font (size 1 1)) (justify left))
     )
-    (property "Footprint" "CEDCp:Resistencia_0,25W" (id 2) (at 130.8862 113.284 0)
+    (property "Footprint" "CEDCp_V2:Resistencia_0,25W" (id 2) (at 130.8862 113.284 0)
       (effects (font (size 1.27 1.27)) hide)
     )
@@
   (symbol (lib_id "Device:R_Small") (at 130.8862 120.904 90) (unit 1)
     (in_bom yes) (on_board yes)
-    (property "Reference" "R34" (id 0) (at 132.1562 118.999 90)
+    (property "Reference" "R35" (id 0) (at 132.1562 118.999 90)
       (effects (font (size 1.27 1.27)) (justify left))
     )
@@
       (effects (font (size 1 1)) (justify left))
     )
-    (property "Footprint" "CEDCp:Resistencia_0,25W" (id 2) (at 130.8862 120.904 0)
+    (property "Footprint" "CEDCp_V2:Resistencia_0,25W" (id 2) (at 130.8862 120.904 0)
       (effects (font (size 1.27 1.27)) hide)
     )
@@
   (symbol (lib_id "Device:R_Potentiometer") (at 154.7622 105.156 0) (unit 1)
     (in_bom yes) (on_board yes)
-    (property "Reference" "RV8" (id 0) (at 159.893 107.188 0)
+    (property "Reference" "U11" (id 0) (at 159.893 107.188 0)
       (effects (font (size 1.27 1.27)) (justify right))
     )
