File: Proteccion Sobre Tension (53V).kicad_sch (KiCad schematic)
At the start: 5 parts, among them K4 SLA-12VDC-SL-C, U16 Fuse

Commit message: Reorder conection with control module
Connections:
- net F_In: now reaches K4.NC, U16.2
Changed lines of the file:
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@@
     (effects (font (size 2 2) (thickness 0.4) bold) (justify left bottom))
+  )
+  (label "F_In" (at 154.5336 146.05 0)
+    (effects (font (size 1.27 1.27)) (justify left bottom))
   )
   (label "3.5V" (at 133.35 71.12 0)

Commit message: Pads mas grandes y correccion de vias
Parts:
- U16: footprint Fuse:Fuse_Littelfuse-LVR100 -> CEDCp:Fuse
Connections:
- net F_In: now also K4.NO; no longer K4.NC
- net GND: no longer K4.NO
- no-connect marks 2 -> 3
Other:
- note removed: "fromuC_PowerEnable: Entrada digital generada por el micro que como maximo tendra 3.3V. Se emplea para habilitar la conexion con el dispositivo bajo prueba (proteccion por sobre tension)."
Changed lines of the file:
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@@
   (junction (at 172.72 66.04) (diameter 0) (color 0 0 0 0)
   )
+  (no_connect (at 148.59 143.51))
   (no_connect (at 152.4 81.28))
   (no_connect (at 154.94 81.28))
@@
     (stroke (width 0) (type default) (color 0 0 0 0))
   )
-  (wire (pts (xy 163.83 146.05) (xy 148.59 146.05))
+  (wire (pts (xy 138.43 146.05) (xy 163.83 146.05))
     (stroke (width 0) (type default) (color 0 0 0 0))
   )
@@
     (stroke (width 0) (type default) (color 0 0 0 0))
   )
-  (wire (pts (xy 149.86 90.17) (xy 105.41 90.17))
+  (wire (pts (xy 138.43 146.05) (xy 138.43 143.51))
     (stroke (width 0) (type default) (color 0 0 0 0))
   )
-  (wire (pts (xy 148.59 146.05) (xy 148.59 143.51))
+  (wire (pts (xy 149.86 90.17) (xy 105.41 90.17))
     (stroke (width 0) (type default) (color 0 0 0 0))
   )
@@
     (effects (font (size 2.9972 2.9972) (thickness 0.5994) bold) (justify left bottom))
   )
-  (text "fromuC_PowerEnable: Entrada digital generada \npor el micro que como maximo tendra 3.3V. \nSe emplea para habilitar la conexion \ncon el dispositivo bajo prueba \n(proteccion por sobre tension)."
-    (at 39.624 128.016 0)
-    (effects (font (size 1.4986 1.4986) (thickness 0.2997) bold) (justify left bottom))
-  )
   (text "uC_OverVoltage:  Señal de 3.3V que se conecta \ndirectamente al uC. Cuando es 1 (3.3V) indica al micro\nque la tension a superado los 53V por tanto debe\ndesconectar la potencia rapidamente."
     (at 214.503 69.469 0)
@@
   (hierarchical_label "+3.3V" (shape input) (at 160.02 73.66 0)
     (effects (font (size 1.2954 1.2954) (thickness 0.2591) bold italic) (justify left))
-  )
-  (hierarchical_label "GND" (shape input) (at 138.43 143.51 180)
-    (effects (font (size 1.2954 1.2954) (thickness 0.2591) bold italic) (justify right))
   )
   (hierarchical_label "VI_3.3V" (shape input) (at 140.97 76.2 180)
@@
     (property "Reference" "U16" (id 0) (at 167.64 141.0462 90))
     (property "Value" "Fuse" (id 1) (at 167.64 143.3576 90))
-    (property "Footprint" "Fuse:Fuse_Littelfuse-LVR100" (id 2) (at 167.64 144.272 90)
+    (property "Footprint" "CEDCp:Fuse" (id 2) (at 167.64 144.272 90)
       (effects (font (size 1.27 1.27)) hide)
     )

Commit message: V4 Ltspice
Parts:
- removed UA1: LM311, CEDCp:LM311P, symbol Comparator:LM311
- added UA1: LM311_V2, CEDCp_V2:LM311_V2, symbol CEDCp_V2:LM311_V2
- R33: renamed from R39; footprint CEDCp:Resistencia_0,25W -> CEDCp_V2:Resistencia_0,25W
- renumbered U16 to U19
Connections:
- net +12V1: now also UA1.8 (V+)
- net +3.3V: now also UA1.7 (COut)
- net 3.5V: now also UA1.3 (-)
- net GND: now also UA1.4 (V-)
- net VI_3.3V: now also UA1.2 (+)
- net toMicroC_OverVoltageSignal: now also UA1.1 (EOut)
Changed lines of the file:
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@@
   (symbol (lib_id "Device:Fuse") (at 167.64 146.05 270) (unit 1)
     (in_bom yes) (on_board yes)
-    (property "Reference" "U16" (id 0) (at 167.64 141.0462 90))
+    (property "Reference" "U19" (id 0) (at 167.64 141.0462 90))
     (property "Value" "Fuse" (id 1) (at 167.64 143.3576 90))
     (property "Footprint" "CEDCp:Fuse" (id 2) (at 167.64 144.272 90)
@@
     (pin "1")
     (pin "2")
-  )
-  (symbol (lib_id "Comparator:LM311") (at 152.4 73.66 0) (mirror x) (unit 1)
-    (in_bom yes) (on_board yes)
-    (property "Reference" "UA1" (id 0) (at 154.94 71.12 0)
-      (effects (font (size 1.27 1.27)) (justify left))
-    )
-    (property "Value" "LM311" (id 1) (at 156.21 76.2 0)
-      (effects (font (size 1.27 1.27)) (justify left))
-    )
-    (property "Footprint" "CEDCp:LM311P" (id 2) (at 152.4 73.66 0)
-      (effects (font (size 1.27 1.27)) hide)
-    )
-    (property "Datasheet" "https://www.st.com/resource/en/datasheet/lm311.pdf" (id 3) (at 152.4 73.66 0)
-      (effects (font (size 1.27 1.27)) hide)
-    )
-    (pin "1")
-    (pin "2")
-    (pin "3")
-    (pin "4")
-    (pin "5")
-    (pin "6")
-    (pin "7")
-    (pin "8")
   )
   (symbol (lib_id "CEDCp:SLA-12VDC-SL-C") (at 143.51 133.35 270) (unit 1)
@@
     (in_bom yes) (on_board yes)
     (property "Reference" "RV10" (id 0) (at 128.4732 73.2282 0)
-      (effects (font (size 1.27 1.27)) (justify right) hide)
+      (effects (font (size 1.27 1.27)) (justify right))
     )
     (property "Value" "5k" (id 1) (at 121.92 70.231 90)
@@
   (symbol (lib_id "Device:R_Small") (at 172.72 73.66 0) (unit 1)
     (in_bom yes) (on_board yes)
-    (property "Reference" "R39" (id 0) (at 173.99 73.66 0)
+    (property "Reference" "R33" (id 0) (at 173.99 73.66 0)
       (effects (font (size 1.27 1.27)) (justify left))
     )
@@
       (effects (font (size 1 1)) (justify left))
     )
-    (property "Footprint" "CEDCp:Resistencia_0,25W" (id 2) (at 172.72 73.66 0)
+    (property "Footprint" "CEDCp_V2:Resistencia_0,25W" (id 2) (at 172.72 73.66 0)
       (effects (font (size 1.27 1.27)) hide)
     )
@@
     (pin "2")
   )
+  (symbol (lib_id "CEDCp_V2:LM311_V2") (at 152.4 73.66 0) (mirror x) (unit 1)
+    (in_bom yes) (on_board yes) (fields_autoplaced)
+    (property "Reference" "UA1" (id 0) (at 164.1602 67.8305 0))
+    (property "Value" "LM311_V2" (id 1) (at 164.1602 70.3705 0))
+    (property "Footprint" "CEDCp_V2:LM311_V2" (id 2) (at 152.4 73.66 0)
+      (effects (font (size 1.27 1.27)) hide)
+    )
+    (property "Datasheet" "https://www.st.com/resource/en/datasheet/lm311.pdf" (id 3) (at 152.4 43.18 0)
+      (effects (font (size 1.27 1.27)) hide)
+    )
+    (pin "1")
+    (pin "2")
+    (pin "3")
+    (pin "4")
+    (pin "5")
+    (pin "6")
+    (pin "7")
+    (pin "8")
+  )
 )
