File: Adaptación_Señal_Control.kicad_sch (KiCad schematic)
At the start: 21 parts, among them Q1 BC337, Q2 BC327, U1 OPA604, U2 OPA604

Commit message: Gerbers generated again
Connections:
- net PushPullOUT: now also U2.2 (-In)
Changed lines of the file:
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@@
   (junction (at 151.511 107.9246) (diameter 0) (color 0 0 0 0)
   )
+  (junction (at 251.8156 100.33) (diameter 0) (color 0 0 0 0)
+  )
   (junction (at 113.03 115.57) (diameter 0) (color 0 0 0 0)
   )
@@
   )
   (junction (at 225.044 91.0844) (diameter 0) (color 0 0 0 0)
-  )
-  (junction (at 249.555 100.33) (diameter 0) (color 0 0 0 0)
   )
   (junction (at 113.03 107.95) (diameter 0) (color 0 0 0 0)
@@
     (stroke (width 0) (type default) (color 0 0 0 0))
   )
-  (wire (pts (xy 249.555 74.93) (xy 249.555 100.33))
-    (stroke (width 0) (type default) (color 0 0 0 0))
-  )
   (wire (pts (xy 244.475 114.3) (xy 244.475 115.57))
     (stroke (width 0) (type default) (color 0 0 0 0))
@@
     (stroke (width 0) (type default) (color 0 0 0 0))
   )
+  (wire (pts (xy 215.8238 95.25) (xy 215.8238 73.8124))
+    (stroke (width 0) (type default) (color 0 0 0 0))
+  )
   (wire (pts (xy 74.93 113.03) (xy 67.31 113.03))
     (stroke (width 0) (type default) (color 0 0 0 0))
@@
     (stroke (width 0) (type default) (color 0 0 0 0))
   )
-  (wire (pts (xy 249.555 100.33) (xy 258.445 100.33))
-    (stroke (width 0) (type default) (color 0 0 0 0))
-  )
   (wire (pts (xy 151.511 109.1946) (xy 151.511 107.9246))
     (stroke (width 0) (type default) (color 0 0 0 0))
@@
     (stroke (width 0) (type default) (color 0 0 0 0))
   )
+  (wire (pts (xy 244.475 100.33) (xy 251.8156 100.33))
+    (stroke (width 0) (type default) (color 0 0 0 0))
+  )
   (wire (pts (xy 236.855 91.44) (xy 236.855 97.79))
     (stroke (width 0) (type default) (color 0 0 0 0))
@@
     (stroke (width 0) (type default) (color 0 0 0 0))
   )
-  (wire (pts (xy 214.5538 74.93) (xy 249.555 74.93))
+  (wire (pts (xy 215.8238 73.8124) (xy 251.8156 73.8124))
     (stroke (width 0) (type default) (color 0 0 0 0))
   )
@@
     (stroke (width 0) (type default) (color 0 0 0 0))
   )
-  (wire (pts (xy 219.0496 95.25) (xy 214.5538 95.25))
-    (stroke (width 0) (type default) (color 0 0 0 0))
-  )
   (wire (pts (xy 125.73 97.79) (xy 128.27 97.79))
     (stroke (width 0) (type default) (color 0 0 0 0))
@@
     (stroke (width 0) (type default) (color 0 0 0 0))
   )
+  (wire (pts (xy 251.8156 100.33) (xy 258.445 100.33))
+    (stroke (width 0) (type default) (color 0 0 0 0))
+  )
   (wire (pts (xy 155.829 93.1926) (xy 152.019 93.1926))
     (stroke (width 0) (type default) (color 0 0 0 0))
   )
+  (wire (pts (xy 251.8156 73.8124) (xy 251.8156 100.33))
+    (stroke (width 0) (type default) (color 0 0 0 0))
+  )
   (wire (pts (xy 74.93 102.87) (xy 67.31 102.87))
     (stroke (width 0) (type default) (color 0 0 0 0))
@@
     (stroke (width 0) (type default) (color 0 0 0 0))
   )
-  (wire (pts (xy 214.5538 95.25) (xy 214.5538 74.93))
-    (stroke (width 0) (type default) (color 0 0 0 0))
-  )
   (wire (pts (xy 138.43 75.692) (xy 138.43 97.79))
     (stroke (width 0) (type default) (color 0 0 0 0))
@@
     (stroke (width 0) (type default) (color 0 0 0 0))
   )
+  (wire (pts (xy 219.075 95.25) (xy 215.8238 95.25))
+    (stroke (width 0) (type default) (color 0 0 0 0))
+  )
   (wire (pts (xy 157.48 75.692) (xy 158.75 75.692))
     (stroke (width 0) (type default) (color 0 0 0 0))
@@
     (stroke (width 0) (type default) (color 0 0 0 0))
   )
-  (wire (pts (xy 244.475 100.33) (xy 249.555 100.33))
-    (stroke (width 0) (type default) (color 0 0 0 0))
-  )

Commit message: Version V1 (Clearence + pads)
Parts:
- D1: value 1N47xxA -> BZX384B3V9
- R2: value 2k7 -> 1k2
- UB1: value 74HC4051N,652 -> 74HC4051N
Changed lines of the file:
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@@
       (effects (font (size 1.27 1.27)) (justify left))
     )
-    (property "Value" "1N47xxA" (id 1) (at 200.787 109.093 90)
+    (property "Value" "BZX384B3V9" (id 1) (at 200.787 109.093 90)
       (effects (font (size 1.27 1.27)) (justify left))
     )
@@
     (in_bom yes) (on_board yes)
     (property "Reference" "UB1" (id 0) (at 92.71 88.392 0))
-    (property "Value" "74HC4051N,652" (id 1) (at 92.71 90.7034 0))
+    (property "Value" "74HC4051N" (id 1) (at 92.71 90.7034 0))
     (property "Footprint" "CEDCp:74HC4051M" (id 2) (at 92.71 107.95 0)
       (effects (font (size 1.27 1.27)) (justify left bottom) hide)
@@
       (effects (font (size 1.27 1.27)) (justify left))
     )
-    (property "Value" "2k7" (id 1) (at 59.7408 116.84 90)
-      (effects (font (size 1 1)) (justify left))
-    )
+    (property "Value" "1k2" (id 1) (at 59.7408 116.84 90)
+      (effects (font (size 1 1)) (justify left))
+    )

Commit message: Heat sink added + Large pads
Other:
- note added: "8-channel analog multiplexer/demultiplexer"
- note added: "En este caso esta funcionando como un multiplexor, uniendo las señales de error a la señal de salida."
Changed lines of the file:
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@@
     (effects (font (size 1.4986 1.4986) (thickness 0.2997) bold) (justify left bottom))
+  )
+  (text "8-channel analog multiplexer/demultiplexer" (at 75.1078 138.557 0)
+    (effects (font (size 1.27 1.27)) (justify left bottom))
   )
   (text "R4, R14, R5 y R7 con tolerancia del 1%" (at 60.579 66.929 0)
@@
     (effects (font (size 1.4986 1.4986) (thickness 0.2997) bold) (justify left bottom))
   )
+  (text "En este caso esta funcionando como un multiplexor, \nuniendo las señales de error a la señal de salida."
+    (at 74.2442 144.4752 0)
+    (effects (font (size 1.27 1.27)) (justify left bottom))
+  )
   (label "PushPullIN" (at 202.565 100.33 0)

Commit message: Pads mas grandes y correccion de vias
Connections:
- net fromMicroC_FeedbackLoopSelection renamed fromA6841_FeedbackLoopSelection
Changed lines of the file:
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@@
     (effects (font (size 1.2954 1.2954) (thickness 0.2591) bold italic) (justify left))
   )
-  (hierarchical_label "fromMicroC_FeedbackLoopSelection" (shape input) (at 58.42 107.95 180)
+  (hierarchical_label "fromA6841_FeedbackLoopSelection" (shape input) (at 58.42 107.95 180)
     (effects (font (size 1.2954 1.2954) (thickness 0.2591) bold italic) (justify right))
   )

Commit message: V4 Ltspice
Parts:
- D5: renamed from D1; footprint Diode_THT:D_DO-15_P10.16mm_Horizontal -> Diode_THT:D_DO-41_SOD81_P10.16mm_Horizontal
- Q61: renamed from Q1; footprint CEDCp:BC548 -> Package_TO_SOT_THT:TO-92_Inline
- Q62: renamed from Q2; footprint CEDCp:BC548 -> Package_TO_SOT_THT:TO-92_Inline
- R14: renamed from R4; footprint CEDCp:Resistencia_0,25W -> CEDCp_V2:Resistencia_0,25W
- R3: renamed from R7; footprint CEDCp:Resistencia_0,25W -> CEDCp_V2:Resistencia_0,25W
- R4: renamed from R3; footprint CEDCp:Resistencia_0,25W -> CEDCp_V2:Resistencia_0,25W
- R5: footprint CEDCp:Resistencia_0,25W -> CEDCp_V2:Resistencia_0,25W
- R6: renamed from R1; footprint CEDCp:Resistencia_0,25W -> CEDCp_V2:Resistencia_0,25W
- R7: renamed from R6; footprint CEDCp:Resistencia_0,25W -> CEDCp_V2:Resistencia_0,25W
- R9: renamed from R2; footprint CEDCp:Resistencia_0,25W -> CEDCp_V2:Resistencia_0,25W
- renumbered C8 to C2, C7 to C28, C6 to C29, C11 to C30, C10 to C31, C9 to C4, U1 to U6, U2 to U60, UB1 to UB3
Connections:
- net -12V: now also Q62.1 (C); no longer Q62.3 (E)
- net PushPullOUT: now also Q62.3 (E); no longer Q62.1 (C)

Commit message: VF4 actualizaciones
Other:
- note added: "Resistencias de offset 250k en vez de 100k Capacitores de desacople.."
Changed lines of the file:
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@@
     (effects (font (size 1.4986 1.4986) (thickness 0.2997) bold) (justify left bottom))
+  )
+  (text "Resistencias de offset 250k en vez de 100k\nCapacitores de desacople.."
+    (at 206.7814 51.2826 0)
+    (effects (font (size 3 3) bold italic) (justify left bottom))
   )
   (text "C30 y C31 son capacitores de tantalio.Deben conectarse\nlo mas cerca posible de los pines de alimentacion del U60"
